File: Board Schematics/Possible board Schematic.sch (EAGLE design)
At the start: 21 parts

Commit message: Started Board Schemate
Parts:
- removed FID1, FID2: FIDUCIAL_1MM, microbuilder:FIDUCIAL_1MM
- removed R2: 10K, microbuilder:RESISTOR_4PACK
Connections:
- removed net A0: R5G$2.2, U$1.A0
- removed net A1: R5G$1.2, U$1.A1
- removed net A2: R2G$1.2, U$5.A0
- net GND: now also U$1.A0, U$1.A1, U$5.A0; no longer R2G$1.1, R5G$1.1, R5G$2.1
Changed lines of the file:
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@@
 <part name="GND3" library="supply1" library_urn="urn:adsk.eagle:library:371" deviceset="GND" device=""/>
 <part name="JP1" library="microbuilder" deviceset="HEADER-1X4" device="ROUND"/>
-<part name="GND4" library="supply1" library_urn="urn:adsk.eagle:library:371" deviceset="GND" device=""/>
-<part name="GND5" library="supply1" library_urn="urn:adsk.eagle:library:371" deviceset="GND" device=""/>
 <part name="U$2" library="microbuilder" deviceset="MOUNTINGHOLE" device="2.5"/>
 <part name="U$3" library="microbuilder" deviceset="MOUNTINGHOLE" device="2.5"/>
 <part name="R5" library="microbuilder" deviceset="RESISTOR_4PACK" device="" value="10K"/>
 <part name="U$4" library="microbuilder" deviceset="FRAME_A4_ADAFRUIT" device=""/>
-<part name="FID1" library="microbuilder" deviceset="FIDUCIAL" device="_1MM"/>
-<part name="FID2" library="microbuilder" deviceset="FIDUCIAL" device="_1MM"/>
 <part name="SJ3" library="microbuilder" deviceset="SOLDERJUMPER" device="CLOSED"/>
 <part name="U$6" library="microbuilder" deviceset="MOUNTINGHOLE" device="2.5"/>
@@
 <part name="GND9" library="supply1" library_urn="urn:adsk.eagle:library:371" deviceset="GND" device=""/>
 <part name="P+9" library="supply1" library_urn="urn:adsk.eagle:library:371" deviceset="VCC" device=""/>
-<part name="GND1" library="supply1" library_urn="urn:adsk.eagle:library:371" deviceset="GND" device=""/>
-<part name="R2" library="microbuilder" deviceset="RESISTOR_4PACK" device="" value="10K"/>
 <part name="JP3" library="microbuilder" deviceset="HEADER-1X4" device="ROUND"/>
 <part name="JP4" library="microbuilder" deviceset="HEADER-1X4" device="ROUND"/>
@@
 <attribute name="VALUE" x="179.07" y="104.14" size="1.778" layer="96"/>
 </instance>
-<instance part="GND4" gate="1" x="17.78" y="106.68" smashed="yes">
-<attribute name="VALUE" x="15.24" y="104.14" size="1.778" layer="96"/>
-</instance>
-<instance part="GND5" gate="1" x="27.94" y="106.68" smashed="yes">
-<attribute name="VALUE" x="25.4" y="104.14" size="1.778" layer="96"/>
-</instance>
 <instance part="U$2" gate="G$1" x="185.42" y="-17.78" smashed="yes"/>
 <instance part="U$3" gate="G$1" x="185.42" y="-10.16" smashed="yes"/>
-<instance part="R5" gate="G$1" x="27.94" y="116.84" smashed="yes" rot="R90">
-<attribute name="NAME" x="25.4" y="116.84" size="1.27" layer="95" font="vector" rot="R90" align="center"/>
-<attribute name="VALUE" x="27.94" y="116.84" size="1.016" layer="96" font="vector" ratio="15" rot="R90" align="center"/>
-</instance>
-<instance part="R5" gate="G$2" x="17.78" y="116.84" smashed="yes" rot="R90">
-<attribute name="NAME" x="15.24" y="116.84" size="1.27" layer="95" font="vector" rot="R90" align="center"/>
-<attribute name="VALUE" x="17.78" y="116.84" size="1.016" layer="96" font="vector" ratio="15" rot="R90" align="center"/>
-</instance>
 <instance part="R5" gate="G$3" x="53.34" y="114.3" smashed="yes" rot="R90">
 <attribute name="NAME" x="50.8" y="114.3" size="1.27" layer="95" font="vector" rot="R90" align="center"/>
@@
 <attribute name="SHEET" x="172.085" y="-30.48" size="2.54" layer="94" font="vector"/>
 </instance>
-<instance part="FID1" gate="G$1" x="177.8" y="-17.78" smashed="yes"/>
-<instance part="FID2" gate="G$1" x="177.8" y="-10.16" smashed="yes"/>
 <instance part="SJ3" gate="1" x="15.24" y="43.18" smashed="yes">
 <attribute name="NAME" x="12.7" y="45.72" size="1.27" layer="95"/>
@@
 <attribute name="VALUE" x="-20.32" y="121.92" size="1.778" layer="96" rot="R90"/>
 </instance>
-<instance part="GND1" gate="1" x="35.56" y="106.68" smashed="yes">
-<attribute name="VALUE" x="33.02" y="104.14" size="1.778" layer="96"/>
-</instance>
-<instance part="R2" gate="G$1" x="35.56" y="116.84" smashed="yes" rot="R90">
-<attribute name="NAME" x="33.02" y="116.84" size="1.27" layer="95" font="vector" rot="R90" align="center"/>
-<attribute name="VALUE" x="35.56" y="116.84" size="1.016" layer="96" font="vector" ratio="15" rot="R90" align="center"/>
-</instance>
 <instance part="JP3" gate="A" x="104.14" y="111.76" smashed="yes">
 <attribute name="NAME" x="97.79" y="120.015" size="1.778" layer="95"/>
@@
 </segment>
 <segment>
-<pinref part="GND5" gate="1" pin="GND"/>
-<pinref part="R5" gate="G$1" pin="1"/>
-<wire x1="27.94" y1="109.22" x2="27.94" y2="111.76" width="0.1524" layer="91"/>
-</segment>
-<segment>
-<pinref part="GND4" gate="1" pin="GND"/>
-<pinref part="R5" gate="G$2" pin="1"/>
-<wire x1="17.78" y1="109.22" x2="17.78" y2="111.76" width="0.1524" layer="91"/>
-</segment>
-<segment>
 <pinref part="R1" gate="G$1" pin="2"/>
 <pinref part="GND6" gate="1" pin="GND"/>
@@
 </segment>
 <segment>
-<pinref part="GND1" gate="1" pin="GND"/>
-<pinref part="R2" gate="G$1" pin="1"/>
-<wire x1="35.56" y1="109.22" x2="35.56" y2="111.76" width="0.1524" layer="91"/>
-</segment>
-<segment>
 <pinref part="JP4" gate="A" pin="2"/>
 <wire x1="129.54" y1="114.3" x2="116.84" y2="114.3" width="0.1524" layer="91"/>
@@
 <wire x1="157.48" y1="116.84" x2="144.78" y2="116.84" width="0.1524" layer="91"/>
 <label x="144.78" y="116.84" size="1.778" layer="95"/>
+</segment>
+<segment>
+<pinref part="U$1" gate="G$1" pin="A1"/>
+<wire x1="-27.94" y1="43.18" x2="-33.02" y2="43.18" width="0.1524" layer="91"/>
+<label x="-33.02" y="43.18" size="1.778" layer="95"/>
+</segment>
+<segment>
+<pinref part="U$1" gate="G$1" pin="A0"/>
+<wire x1="-27.94" y1="40.64" x2="-33.02" y2="40.64" width="0.1524" layer="91"/>
+<label x="-33.02" y="40.64" size="1.778" layer="95"/>
+</segment>
+<segment>
+<pinref part="U$5" gate="G$1" pin="A0"/>
+<wire x1="58.42" y1="40.64" x2="53.34" y2="40.64" width="0.1524" layer="91"/>
+<label x="53.34" y="40.64" size="1.778" layer="95"/>
 </segment>
 </net>
@@
 <wire x1="157.48" y1="119.38" x2="144.78" y2="119.38" width="0.1524" layer="91"/>
 <label x="144.78" y="119.38" size="1.778" layer="95"/>
-</segment>
-</net>
-<net name="A0" class="0">
-<segment>
-<pinref part="U$1" gate="G$1" pin="A0"/>
-<wire x1="-27.94" y1="40.64" x2="-33.02" y2="40.64" width="0.1524" layer="91"/>
-<label x="-33.02" y="40.64" size="1.778" layer="95"/>
-</segment>
-<segment>
-<wire x1="17.78" y1="121.92" x2="17.78" y2="124.46" width="0.1524" layer="91"/>
-<label x="15.24" y="124.46" size="1.778" layer="95"/>
-<pinref part="R5" gate="G$2" pin="2"/>
-</segment>
-</net>
-<net name="A1" class="0">
-<segment>
-<pinref part="U$1" gate="G$1" pin="A1"/>
-<wire x1="-27.94" y1="43.18" x2="-33.02" y2="43.18" width="0.1524" layer="91"/>
-<label x="-33.02" y="43.18" size="1.778" layer="95"/>
-</segment>
-<segment>
-<wire x1="27.94" y1="121.92" x2="27.94" y2="124.46" width="0.1524" layer="91"/>
-<label x="25.4" y="124.46" size="1.778" layer="95"/>
-<pinref part="R5" gate="G$1" pin="2"/>
 </segment>
 </net>
@@
 </segment>
 </net>
-<net name="A2" class="0">
-<segment>
-<pinref part="U$5" gate="G$1" pin="A0"/>
-<wire x1="58.42" y1="40.64" x2="53.34" y2="40.64" width="0.1524" layer="91"/>
-<label x="53.34" y="40.64" size="1.778" layer="95"/>
-</segment>
-<segment>
-<wire x1="35.56" y1="121.92" x2="35.56" y2="124.46" width="0.1524" layer="91"/>
-<label x="33.02" y="124.46" size="1.778" layer="95"/>
-<pinref part="R2" gate="G$1" pin="2"/>
-</segment>
-</net>
